File: KiCad_Project/RadioTelescope.kicad_sch (KiCad schematic)
At the start: 40 parts, among them J1 Conn_02x19_Odd_Even, J2 Conn_02x19_Odd_Even, J3 Conn_01x01, P1 USB_C_Plug_USB2.0, Q1 BC546, Q2 BC546, Q3 BC546, U1 CH340T, U2 MAX232, Y1 12MHz

Commit message: Added gitignore and added more info to readme
Other:
- title: (none) -> Radio Image Telescope
Changed lines of the file:
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@@
 	(generator_version "9.0")
 	(paper "A3")
+	(title_block
+		(title "Radio Image Telescope")
+		(rev "1")
+	)
 	(text "Red   - Error\nBlue  - Calibrating\nGreen - Ready for Input\nBlue rapidly blinking  - Processening\nGreen rapidly blinking - Running Scan"
 		(exclude_from_sim no)
